Commit message: Add stable surface-aware Go2 leg animation

File: src/caddie_description/urdf/go2_caddie_official.urdf.xacro (robot description, xacro)
@@ -4,4 +4,7 @@
   <xacro:arg name="leg_joint_type" default="fixed"/>
   <xacro:arg name="use_leg_control" default="false"/>
+  <xacro:arg name="use_leg_collision" default="true"/>
+  <xacro:arg name="leg_mass_scale" default="1.0"/>
+  <xacro:property name="leg_mass_scale_value" value="$(arg leg_mass_scale)"/>
   <xacro:macro name="leg_position_joint" params="joint_name lower upper initial">
     <joint name="${joint_name}">
@@ -17,4 +20,10 @@
     </joint>
   </xacro:macro>
+  <xacro:macro name="visual_only_leg_link" params="link_name">
+    <gazebo reference="${link_name}">
+      <gravity>false</gravity>
+      <self_collide>false</self_collide>
+    </gazebo>
+  </xacro:macro>
   <!--
     Base Go2 geometry, inertials, and joint layout are derived from Unitree's
@@ -88,6 +97,6 @@
     <inertial>
       <origin xyz="-0.0054 0.00194 -0.000105" rpy="0 0 0" />
-      <mass value="0.678" />
-      <inertia ixx="0.00048" ixy="-3.01E-06" ixz="1.11E-06" iyy="0.000884" iyz="-1.42E-06" izz="0.000596" />
+      <mass value="${0.678 * float(leg_mass_scale_value)}" />
+      <inertia ixx="${0.00048 * float(leg_mass_scale_value)}" ixy="${-3.01E-06 * float(leg_mass_scale_value)}" ixz="${1.11E-06 * float(leg_mass_scale_value)}" iyy="${0.000884 * float(leg_mass_scale_value)}" iyz="${-1.42E-06 * float(leg_mass_scale_value)}" izz="${0.000596 * float(leg_mass_scale_value)}" />
     </inertial>
     <visual>
@@ -97,4 +106,5 @@
       </geometry>
       <material name="深色橡胶_001-effect"><color rgba="0.6717055 0.6924257 0.7742702 1" /></material><material name="Material-effect"><color rgba="0.9 0.95 0.95 1" /></material></visual>
+    <xacro:if value="$(arg use_leg_collision)">
     <collision>
       <origin rpy="1.5707963267948966 0 0" xyz="0 0.08 0" />
@@ -103,4 +113,5 @@
       </geometry>
     </collision>
+    </xacro:if>
   </link>
   <joint name="FL_hip_joint" type="$(arg leg_joint_type)">
@@ -126,6 +137,6 @@
     <inertial>
       <origin xyz="-0.00374 -0.0223 -0.0327" rpy="0 0 0" />
-      <mass value="1.152" />
-      <inertia ixx="0.00584" ixy="8.72E-05" ixz="-0.000289" iyy="0.0058" iyz="0.000808" izz="0.00103" />
+      <mass value="${1.152 * float(leg_mass_scale_value)}" />
+      <inertia ixx="${0.00584 * float(leg_mass_scale_value)}" ixy="${8.72E-05 * float(leg_mass_scale_value)}" ixz="${-0.000289 * float(leg_mass_scale_value)}" iyy="${0.0058 * float(leg_mass_scale_value)}" iyz="${0.000808 * float(leg_mass_scale_value)}" izz="${0.00103 * float(leg_mass_scale_value)}" />
     </inertial>
     <visual>
@@ -135,4 +146,5 @@
       </geometry>
       <material name="深色橡胶_003-effect"><color rgba="0.6717055 0.6924257 0.7742702 1" /></material><material name="Material_009-effect"><color rgba="0.9 0.95 0.95 1" /></material></visual>
+    <xacro:if value="$(arg use_leg_collision)">
     <collision>
       <origin rpy="0 1.5707963267948966 0" xyz="0 0 -0.1065" />
@@ -141,4 +153,5 @@
       </geometry>
     </collision>
+    </xacro:if>
   </link>
   <joint name="FL_thigh_joint" type="$(arg leg_joint_type)">
@@ -164,6 +177,6 @@
     <inertial>
       <origin xyz="0.00548 -0.000975 -0.115" rpy="0 0 0" />
-      <mass value="0.154" />
-      <inertia ixx="0.00108" ixy="3.4E-07" ixz="1.72E-05" iyy="0.0011" iyz="8.28E-06" izz="3.29E-05" />
+      <mass value="${0.154 * float(leg_mass_scale_value)}" />
+      <inertia ixx="${0.00108 * float(leg_mass_scale_value)}" ixy="${3.4E-07 * float(leg_mass_scale_value)}" ixz="${1.72E-05 * float(leg_mass_scale_value)}" iyy="${0.0011 * float(leg_mass_scale_value)}" iyz="${8.28E-06 * float(leg_mass_scale_value)}" izz="${3.29E-05 * float(leg_mass_scale_value)}" />
     </inertial>
     <visual>
@@ -173,4 +186,5 @@
       </geometry>
       <material name="黑色足端_005-effect"><color rgba="0 0 0 1" /></material><material name="深色橡胶_005-effect"><color rgba="0.6717055 0.6924257 0.7742702 1" /></material></visual>
+    <xacro:if value="$(arg use_leg_collision)">
     <collision>
       <origin rpy="0 -0.21 0" xyz="0.008 0 -0.06" />
@@ -179,4 +193,5 @@
       </geometry>
     </collision>
+    </xacro:if>
   </link>
   <joint name="FL_calf_joint" type="$(arg leg_joint_type)">
@@ -188,4 +203,5 @@
   </joint>
   <link name="FL_calflower">
+    <xacro:if value="$(arg use_leg_collision)">
     <collision>
       <origin rpy="0 0 0" xyz="0 0 0" />
@@ -194,4 +210,5 @@
       </geometry>
     </collision>
+    </xacro:if>
   </link>
   <joint name="FL_calflower_joint" type="fixed">
@@ -202,4 +219,5 @@
   </joint>
   <link name="FL_calflower1">
+    <xacro:if value="$(arg use_leg_collision)">
     <collision>
       <origin rpy="0 0 0" xyz="0 0 0" />
@@ -208,4 +226,5 @@
       </geometry>
     </collision>
+    </xacro:if>
   </link>
   <joint name="FL_calflower1_joint" type="fixed">
@@ -230,6 +249,6 @@
     <inertial>
       <origin xyz="0 0 0" rpy="0 0 0" />
-      <mass value="0.04" />
-      <inertia ixx="9.6e-06" ixy="0" ixz="0" iyy="9.6e-06" iyz="0" izz="9.6e-06" />
+      <mass value="${0.04 * float(leg_mass_scale_value)}" />
+      <inertia ixx="${9.6e-06 * float(leg_mass_scale_value)}" ixy="${0 * float(leg_mass_scale_value)}" ixz="${0 * float(leg_mass_scale_value)}" iyy="${9.6e-06 * float(leg_mass_scale_value)}" iyz="${0 * float(leg_mass_scale_value)}" izz="${9.6e-06 * float(leg_mass_scale_value)}" />
     </inertial>
     <visual>
@@ -239,4 +258,5 @@
       </geometry>
       <material name="黑色足端_007-effect"><color rgba="0 0 0 1" /></material></visual>
+    <xacro:if value="$(arg use_leg_collision)">
     <collision>
       <origin rpy="0 0 0" xyz="-0.002 0 0" />
@@ -245,4 +265,5 @@
       </geometry>
     </collision>
+    </xacro:if>
   </link>
   <joint name="FL_foot_joint" type="fixed" dont_collapse="true">
@@ -255,6 +276,6 @@
     <inertial>
       <origin xyz="-0.0054 -0.00194 -0.000105" rpy="0 0 0" />
-      <mass value="0.678" />
-      <inertia ixx="0.00048" ixy="3.01E-06" ixz="1.11E-06" iyy="0.000884" iyz="1.42E-06" izz="0.000596" />
+      <mass value="${0.678 * float(leg_mass_scale_value)}" />
+      <inertia ixx="${0.00048 * float(leg_mass_scale_value)}" ixy="${3.01E-06 * float(leg_mass_scale_value)}" ixz="${1.11E-06 * float(leg_mass_scale_value)}" iyy="${0.000884 * float(leg_mass_scale_value)}" iyz="${1.42E-06 * float(leg_mass_scale_value)}" izz="${0.000596 * float(leg_mass_scale_value)}" />
     </inertial>
     <visual>
@@ -264,4 +285,5 @@
       </geometry>
       <material name="深色橡胶_001-effect"><color rgba="0.6717055 0.6924257 0.7742702 1" /></material><material name="Material-effect"><color rgba="0.9 0.95 0.95 1" /></material></visual>
+    <xacro:if value="$(arg use_leg_collision)">
     <collision>
       <origin rpy="1.5707963267948966 0 0" xyz="0 -0.08 0" />
@@ -270,4 +292,5 @@
       </geometry>
     </collision>
+    </xacro:if>
   </link>
   <joint name="FR_hip_joint" type="$(arg leg_joint_type)">
@@ -293,6 +316,6 @@
     <inertial>
       <origin xyz="-0.00374 0.0223 -0.0327" rpy="0 0 0" />
-      <mass value="1.152" />
-      <inertia ixx="0.00584" ixy="-8.72E-05" ixz="-0.000289" iyy="0.0058" iyz="-0.000808" izz="0.00103" />
+      <mass value="${1.152 * float(leg_mass_scale_value)}" />
+      <inertia ixx="${0.00584 * float(leg_mass_scale_value)}" ixy="${-8.72E-05 * float(leg_mass_scale_value)}" ixz="${-0.000289 * float(leg_mass_scale_value)}" iyy="${0.0058 * float(leg_mass_scale_value)}" iyz="${-0.000808 * float(leg_mass_scale_value)}" izz="${0.00103 * float(leg_mass_scale_value)}" />
     </inertial>
     <visual>
@@ -302,4 +325,5 @@
       </geometry>
       <material name="深色橡胶_012-effect"><color rgba="0.6717055 0.6924257 0.7742702 1" /></material><material name="Material_011-effect"><color rgba="0.9 0.95 0.95 1" /></material></visual>
+    <xacro:if value="$(arg use_leg_collision)">
     <collision>
       <origin rpy="0 1.5707963267948966 0" xyz="0 0 -0.1065" />
@@ -308,4 +332,5 @@
       </geometry>
     </collision>
+    </xacro:if>
   </link>
   <joint name="FR_thigh_joint" type="$(arg leg_joint_type)">
@@ -331,6 +356,6 @@
     <inertial>
       <origin xyz="0.00548 0.000975 -0.115" rpy="0 0 0" />
-      <mass value="0.154" />
-      <inertia ixx="0.00108" ixy="-3.4E-07" ixz="1.72E-05" iyy="0.0011" iyz="-8.28E-06" izz="3.29E-05" />
+      <mass value="${0.154 * float(leg_mass_scale_value)}" />
+      <inertia ixx="${0.00108 * float(leg_mass_scale_value)}" ixy="${-3.4E-07 * float(leg_mass_scale_value)}" ixz="${1.72E-05 * float(leg_mass_scale_value)}" iyy="${0.0011 * float(leg_mass_scale_value)}" iyz="${-8.28E-06 * float(leg_mass_scale_value)}" izz="${3.29E-05 * float(leg_mass_scale_value)}" />
     </inertial>
     <visual>
@@ -340,4 +365,5 @@
       </geometry>
       <material name="黑色足端_006-effect"><color rgba="0 0 0 1" /></material><material name="深色橡胶_007-effect"><color rgba="0.6717055 0.6924257 0.7742702 1" /></material></visual>
+    <xacro:if value="$(arg use_leg_collision)">
     <collision>
       <origin rpy="0 -0.2 0" xyz="0.01 0 -0.06" />
@@ -346,4 +372,5 @@
       </geometry>
     </collision>
+    </xacro:if>
   </link>
   <joint name="FR_calf_joint" type="$(arg leg_joint_type)">
@@ -355,4 +382,5 @@
   </joint>
   <link name="FR_calflower">
+    <xacro:if value="$(arg use_leg_collision)">
     <collision>
       <origin rpy="0 0 0" xyz="0 0 0" />
@@ -361,4 +389,5 @@
       </geometry>
     </collision>
+    </xacro:if>
   </link>
   <joint name="FR_calflower_joint" type="fixed">
@@ -369,4 +398,5 @@
   </joint>
   <link name="FR_calflower1">
+    <xacro:if value="$(arg use_leg_collision)">
     <collision>
       <origin rpy="0 0 0" xyz="0 0 0" />
@@ -375,4 +405,5 @@
       </geometry>
     </collision>
+    </xacro:if>
   </link>
   <joint name="FR_calflower1_joint" type="fixed">
@@ -397,6 +428,6 @@
     <inertial>
       <origin xyz="0 0 0" rpy="0 0 0" />
-      <mass value="0.04" />
-      <inertia ixx="9.6e-06" ixy="0" ixz="0" iyy="9.6e-06" iyz="0" izz="9.6e-06" />
+      <mass value="${0.04 * float(leg_mass_scale_value)}" />
+      <inertia ixx="${9.6e-06 * float(leg_mass_scale_value)}" ixy="${0 * float(leg_mass_scale_value)}" ixz="${0 * float(leg_mass_scale_value)}" iyy="${9.6e-06 * float(leg_mass_scale_value)}" iyz="${0 * float(leg_mass_scale_value)}" izz="${9.6e-06 * float(leg_mass_scale_value)}" />
     </inertial>
     <visual>
@@ -406,4 +437,5 @@
       </geometry>
       <material name="黑色足端_007-effect"><color rgba="0 0 0 1" /></material></visual>
+    <xacro:if value="$(arg use_leg_collision)">
     <collision>
       <origin rpy="0 0 0" xyz="-0.002 0 0" />
@@ -412,4 +444,5 @@
       </geometry>
     </collision>
+    </xacro:if>
   </link>
   <joint name="FR_foot_joint" type="fixed" dont_collapse="true">
@@ -422,6 +455,6 @@
     <inertial>
       <origin xyz="0.0054 0.00194 -0.000105" rpy="0 0 0" />
-      <mass value="0.678" />
-      <inertia ixx="0.00048" ixy="3.01E-06" ixz="-1.11E-06" iyy="0.000884" iyz="-1.42E-06" izz="0.000596" />
+      <mass value="${0.678 * float(leg_mass_scale_value)}" />
+      <inertia ixx="${0.00048 * float(leg_mass_scale_value)}" ixy="${3.01E-06 * float(leg_mass_scale_value)}" ixz="${-1.11E-06 * float(leg_mass_scale_value)}" iyy="${0.000884 * float(leg_mass_scale_value)}" iyz="${-1.42E-06 * float(leg_mass_scale_value)}" izz="${0.000596 * float(leg_mass_scale_value)}" />
     </inertial>
     <visual>
@@ -431,4 +464,5 @@
       </geometry>
       <material name="深色橡胶_001-effect"><color rgba="0.6717055 0.6924257 0.7742702 1" /></material><material name="Material-effect"><color rgba="0.9 0.95 0.95 1" /></material></visual>
+    <xacro:if value="$(arg use_leg_collision)">
     <collision>
       <origin rpy="1.5707963267948966 0 0" xyz="0 0.08 0" />
@@ -437,4 +471,5 @@
       </geometry>
     </collision>
+    </xacro:if>
   </link>
   <joint name="RL_hip_joint" type="$(arg leg_joint_type)">
@@ -460,6 +495,6 @@
     <inertial>
       <origin xyz="-0.00374 -0.0223 -0.0327" rpy="0 0 0" />
-      <mass value="1.152" />
-      <inertia ixx="0.00584" ixy="8.72E-05" ixz="-0.000289" iyy="0.0058" iyz="0.000808" izz="0.00103" />
+      <mass value="${1.152 * float(leg_mass_scale_value)}" />
+      <inertia ixx="${0.00584 * float(leg_mass_scale_value)}" ixy="${8.72E-05 * float(leg_mass_scale_value)}" ixz="${-0.000289 * float(leg_mass_scale_value)}" iyy="${0.0058 * float(leg_mass_scale_value)}" iyz="${0.000808 * float(leg_mass_scale_value)}" izz="${0.00103 * float(leg_mass_scale_value)}" />
     </inertial>
     <visual>
@@ -469,4 +504,5 @@
       </geometry>
       <material name="深色橡胶_003-effect"><color rgba="0.6717055 0.6924257 0.7742702 1" /></material><material name="Material_009-effect"><color rgba="0.9 0.95 0.95 1" /></material></visual>
+    <xacro:if value="$(arg use_leg_collision)">
     <collision>
       <origin rpy="0 1.5707963267948966 0" xyz="0 0 -0.1065" />
@@ -475,4 +511,5 @@
       </geometry>
     </collision>
+    </xacro:if>
   </link>
   <joint name="RL_thigh_joint" type="$(arg leg_joint_type)">
@@ -498,6 +535,6 @@
     <inertial>
       <origin xyz="0.00548 -0.000975 -0.115" rpy="0 0 0" />
-      <mass value="0.154" />
-      <inertia ixx="0.00108" ixy="3.4E-07" ixz="1.72E-05" iyy="0.0011" iyz="8.28E-06" izz="3.29E-05" />
+      <mass value="${0.154 * float(leg_mass_scale_value)}" />
+      <inertia ixx="${0.00108 * float(leg_mass_scale_value)}" ixy="${3.4E-07 * float(leg_mass_scale_value)}" ixz="${1.72E-05 * float(leg_mass_scale_value)}" iyy="${0.0011 * float(leg_mass_scale_value)}" iyz="${8.28E-06 * float(leg_mass_scale_value)}" izz="${3.29E-05 * float(leg_mass_scale_value)}" />
     </inertial>
     <visual>
@@ -507,4 +544,5 @@
       </geometry>
       <material name="黑色足端_005-effect"><color rgba="0 0 0 1" /></material><material name="深色橡胶_005-effect"><color rgba="0.6717055 0.6924257 0.7742702 1" /></material></visual>
+    <xacro:if value="$(arg use_leg_collision)">
     <collision>
       <origin rpy="0 -0.2 0" xyz="0.01 0 -0.06" />
@@ -513,4 +551,5 @@
       </geometry>
     </collision>
+    </xacro:if>
   </link>
   <joint name="RL_calf_joint" type="$(arg leg_joint_type)">
@@ -522,4 +561,5 @@
   </joint>
   <link name="RL_calflower">
+    <xacro:if value="$(arg use_leg_collision)">
     <collision>
       <origin rpy="0 0 0" xyz="0 0 0" />
@@ -528,4 +568,5 @@
       </geometry>
     </collision>
+    </xacro:if>
   </link>
   <joint name="RL_calflower_joint" type="fixed">
@@ -536,4 +577,5 @@
   </joint>
   <link name="RL_calflower1">
+    <xacro:if value="$(arg use_leg_collision)">
     <collision>
       <origin rpy="0 0 0" xyz="0 0 0" />
@@ -542,4 +584,5 @@
       </geometry>
     </collision>
+    </xacro:if>
   </link>
   <joint name="RL_calflower1_joint" type="fixed">
@@ -564,6 +607,6 @@
     <inertial>
       <origin xyz="0 0 0" rpy="0 0 0" />
-      <mass value="0.04" />
-      <inertia ixx="9.6e-06" ixy="0" ixz="0" iyy="9.6e-06" iyz="0" izz="9.6e-06" />
+      <mass value="${0.04 * float(leg_mass_scale_value)}" />
+      <inertia ixx="${9.6e-06 * float(leg_mass_scale_value)}" ixy="${0 * float(leg_mass_scale_value)}" ixz="${0 * float(leg_mass_scale_value)}" iyy="${9.6e-06 * float(leg_mass_scale_value)}" iyz="${0 * float(leg_mass_scale_value)}" izz="${9.6e-06 * float(leg_mass_scale_value)}" />
     </inertial>
     <visual>
@@ -573,4 +616,5 @@
       </geometry>
       <material name="黑色足端_007-effect"><color rgba="0 0 0 1" /></material></visual>
+    <xacro:if value="$(arg use_leg_collision)">
     <collision>
       <origin rpy="0 0 0" xyz="-0.002 0 0" />
@@ -579,4 +623,5 @@
       </geometry>
     </collision>
+    </xacro:if>
   </link>
   <joint name="RL_foot_joint" type="fixed" dont_collapse="true">
@@ -589,6 +634,6 @@
     <inertial>
       <origin xyz="0.0054 -0.00194 -0.000105" rpy="0 0 0" />
-      <mass value="0.678" />
-      <inertia ixx="0.00048" ixy="-3.01E-06" ixz="-1.11E-06" iyy="0.000884" iyz="1.42E-06" izz="0.000596" />
+      <mass value="${0.678 * float(leg_mass_scale_value)}" />
+      <inertia ixx="${0.00048 * float(leg_mass_scale_value)}" ixy="${-3.01E-06 * float(leg_mass_scale_value)}" ixz="${-1.11E-06 * float(leg_mass_scale_value)}" iyy="${0.000884 * float(leg_mass_scale_value)}" iyz="${1.42E-06 * float(leg_mass_scale_value)}" izz="${0.000596 * float(leg_mass_scale_value)}" />
     </inertial>
     <visual>
@@ -598,4 +643,5 @@
       </geometry>
       <material name="深色橡胶_001-effect"><color rgba="0.6717055 0.6924257 0.7742702 1" /></material><material name="Material-effect"><color rgba="0.9 0.95 0.95 1" /></material></visual>
+    <xacro:if value="$(arg use_leg_collision)">
     <collision>
       <origin rpy="1.5707963267948966 0 0" xyz="0 -0.08 0" />
@@ -604,4 +650,5 @@
       </geometry>
     </collision>
+    </xacro:if>
   </link>
   <joint name="RR_hip_joint" type="$(arg leg_joint_type)">
@@ -627,6 +674,6 @@
     <inertial>
       <origin xyz="-0.00374 0.0223 -0.0327" rpy="0 0 0" />
-      <mass value="1.152" />
-      <inertia ixx="0.00584" ixy="-8.72E-05" ixz="-0.000289" iyy="0.0058" iyz="-0.000808" izz="0.00103" />
+      <mass value="${1.152 * float(leg_mass_scale_value)}" />
+      <inertia ixx="${0.00584 * float(leg_mass_scale_value)}" ixy="${-8.72E-05 * float(leg_mass_scale_value)}" ixz="${-0.000289 * float(leg_mass_scale_value)}" iyy="${0.0058 * float(leg_mass_scale_value)}" iyz="${-0.000808 * float(leg_mass_scale_value)}" izz="${0.00103 * float(leg_mass_scale_value)}" />
     </inertial>
     <visual>
@@ -636,4 +683,5 @@
       </geometry>
       <material name="深色橡胶_012-effect"><color rgba="0.6717055 0.6924257 0.7742702 1" /></material><material name="Material_011-effect"><color rgba="0.9 0.95 0.95 1" /></material></visual>
+    <xacro:if value="$(arg use_leg_collision)">
     <collision>
       <origin rpy="0 1.5707963267948966 0" xyz="0 0 -0.1065" />
@@ -642,4 +690,5 @@
       </geometry>
     </collision>
+    </xacro:if>
   </link>
   <joint name="RR_thigh_joint" type="$(arg leg_joint_type)">
@@ -665,6 +714,6 @@
     <inertial>
       <origin xyz="0.00548 0.000975 -0.115" rpy="0 0 0" />
-      <mass value="0.154" />
-      <inertia ixx="0.00108" ixy="-3.4E-07" ixz="1.72E-05" iyy="0.0011" iyz="-8.28E-06" izz="3.29E-05" />
+      <mass value="${0.154 * float(leg_mass_scale_value)}" />
+      <inertia ixx="${0.00108 * float(leg_mass_scale_value)}" ixy="${-3.4E-07 * float(leg_mass_scale_value)}" ixz="${1.72E-05 * float(leg_mass_scale_value)}" iyy="${0.0011 * float(leg_mass_scale_value)}" iyz="${-8.28E-06 * float(leg_mass_scale_value)}" izz="${3.29E-05 * float(leg_mass_scale_value)}" />
     </inertial>
     <visual>
@@ -674,4 +723,5 @@
       </geometry>
       <material name="黑色足端_006-effect"><color rgba="0 0 0 1" /></material><material name="深色橡胶_007-effect"><color rgba="0.6717055 0.6924257 0.7742702 1" /></material></visual>
+    <xacro:if value="$(arg use_leg_collision)">
     <collision>
       <origin rpy="0 -0.2 0" xyz="0.01 0 -0.06" />
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